File: Front/Panel.kicad_pcb (KiCad board)
At the start: 2 copper layers, 95.3 x 67 mm, 10 parts

Commit message: FP fix
Other:
- board text added: "CLAYTUNE - ControlMenu V0.1.1 - By TwinTurbo - JLCJLCJLCJLC"
- board text removed: "CLAYTUNE - ControlMenu V0.1.0 - By TwinTurbo - JLCJLCJLCJLC"
